File: hw/mainBoard/eps32.kicad_sch (KiCad schematic)
At the start: 10 parts, among them SW1 SW_Push, SW2 SW_Push, U1 ESP32-WROOM-E

Commit message: hw - kicad neco
Parts:
- R1: now not fitted
Changed lines of the file:
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@@
   )
   (symbol (lib_id "Device:R") (at 223.52 111.76 90) (unit 1)
-    (in_bom yes) (on_board yes) (dnp no) (fields_autoplaced)
+    (in_bom yes) (on_board yes) (dnp yes) (fields_autoplaced)
     (property "Reference" "R1" (at 223.52 105.41 90)
       (effects (font (size 1.27 1.27)))

Commit message: hw
Parts:
- added C4: 22uF, symbol Device:C
- added C5: 2.2uF, symbol Device:C
- added U4: TLV76133DCYR, SOT_8DCYR_TEX, symbol TLV761:PTLV76118DCYR
Connections:
- net 3V3: now also C5.1, U4.2 (OUTPUT), U4.4 (OUTPUT)
- net GND: now also C4.2, C5.2, U4.1 (GND)
- net IO16 renamed UART2_RX
- net IO17 renamed UART2_TX
- net ~{UART_INT} renamed UART1_RX
- net ~{UART_MODULE_CS} renamed UART1_TX
- net ~{UART_MODULE_RST} renamed IO4
- new net 5.5V: C4.1, U4.3 (INPUT)
Other:
- note added: "Modern version od AMS1117 with soft start"
- moved on the sheet: C1, C2, C3, C6, C7, R1, SW1, SW2

Commit message: hw + blok schema
Connections:
- net 5.5V renamed 5.2V
- net IO21 renamed SDA
- net IO22 renamed SCL
- net IO25 renamed LED_STRIP
Other:
- moved on the sheet: C1, C2, C3, C6, C7, R1, SW1, SW2, U1

Commit message: nejaky hw + teorie + desky
Changed lines of the file:
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@@
 (kicad_sch (version 20230121) (generator eeschema)
   (paper "A4")
+  (bus_alias "UART1" (members "UART1_RX" "UART1_TX"))
+  (bus_alias "UART2" (members "UART2_RX" "UART2_TX"))
   (junction (at 50.8 102.87) (diameter 0) (color 0 0 0 0)
   )
@@
     (effects (font (size 1.27 1.27)) (justify left bottom))
   )
-  (hierarchical_label "UART1" (shape bidirectional) (at 269.24 109.22 0) (fields_autoplaced)
+  (hierarchical_label "{UART1}" (shape bidirectional) (at 269.24 109.22 0) (fields_autoplaced)
     (effects (font (size 1.27 1.27)) (justify left))
   )
-  (hierarchical_label "I2C" (shape bidirectional) (at 269.24 147.32 0) (fields_autoplaced)
+  (hierarchical_label "{I2C}" (shape bidirectional) (at 269.24 147.32 0) (fields_autoplaced)
     (effects (font (size 1.27 1.27)) (justify left))
   )
@@
     (effects (font (size 1.27 1.27)) (justify left))
   )
-  (hierarchical_label "JTAG" (shape bidirectional) (at 269.24 134.62 0) (fields_autoplaced)
+  (hierarchical_label "{JTAG}" (shape bidirectional) (at 269.24 134.62 0) (fields_autoplaced)
     (effects (font (size 1.27 1.27)) (justify left))
   )
-  (hierarchical_label "ESP_PINS_1" (shape bidirectional) (at 269.24 96.52 0) (fields_autoplaced)
+  (hierarchical_label "{ESP_PINS_1}" (shape bidirectional) (at 269.24 96.52 0) (fields_autoplaced)
     (effects (font (size 1.27 1.27)) (justify left))
   )
-  (hierarchical_label "ESP_PINS_2" (shape bidirectional) (at 269.24 88.9 0) (fields_autoplaced)
+  (hierarchical_label "{ESP_PINS_2}" (shape bidirectional) (at 269.24 88.9 0) (fields_autoplaced)
     (effects (font (size 1.27 1.27)) (justify left))
   )
@@
     (effects (font (size 1.27 1.27)) (justify left))
   )
-  (hierarchical_label "UART2" (shape bidirectional) (at 269.24 116.84 0) (fields_autoplaced)
+  (hierarchical_label "{UART2}" (shape bidirectional) (at 269.24 116.84 0) (fields_autoplaced)
     (effects (font (size 1.27 1.27)) (justify left))
   )

Commit message: hw - changed uart2 pins, latex- ridici jednotka
Connections:
- net IO4 is gone; now on net UART2_RX: U1.26 (ADC2_CH0/GPIO4)
- net UART2_RX: no longer R1.2, U1.27 (GPIO16)
- new net IO16: R1.2, U1.27 (GPIO16)
Changed lines of the file:
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@@
     (effects (font (size 1.27 1.27)) (justify left bottom))
   )
-  (label "IO4" (at 243.84 50.8 0) (fields_autoplaced)
+  (label "UART2_RX" (at 243.84 50.8 0) (fields_autoplaced)
     (effects (font (size 1.27 1.27)) (justify left bottom))
   )
@@
     (effects (font (size 1.27 1.27)) (justify left bottom))
   )
-  (label "UART2_RX" (at 243.84 55.88 0) (fields_autoplaced)
+  (label "IO16" (at 243.84 55.88 0) (fields_autoplaced)
     (effects (font (size 1.27 1.27)) (justify left bottom))
   )
@@
     (effects (font (size 1.27 1.27)) (justify left bottom))
   )
-  (label "UART2_RX" (at 58.42 170.18 0) (fields_autoplaced)
+  (label "IO16" (at 58.42 170.18 0) (fields_autoplaced)
     (effects (font (size 1.27 1.27)) (justify left bottom))
   )

Commit message: schematka
Other:
- note added: "BOOT button"
- note added: "RST button"
- moved on the sheet: C1, C2, C3, C5, C6, C7, R1, SW1, SW2, U4

Commit message: drawing layout
Parts:
- C1, C4, C5, C6, C7: footprint (none) -> Capacitor_SMD:C_1206_3216Metric_Pad1.33x1.80mm_HandSolder
- C2: renamed from C3; footprint (none) -> Capacitor_SMD:C_1206_3216Metric_Pad1.33x1.80mm_HandSolder
- C3: renamed from C2; footprint (none) -> Capacitor_SMD:C_1206_3216Metric_Pad1.33x1.80mm_HandSolder
- R1: footprint (none) -> Resistor_SMD:R_0805_2012Metric_Pad1.20x1.40mm_HandSolder
- R2: renamed from R1; footprint (none) -> Resistor_SMD:R_0805_2012Metric_Pad1.20x1.40mm_HandSolder
- SW1, SW2: footprint (none) -> Button_Switch_SMD:SW_SPST_B3U-1000P
Connections:
- net UART2_TX is gone; now on net LED_STRIP: U1.28 (GPIO17)
- net LED_STRIP: no longer U1.10 (DAC_1/ADC2_CH8/GPIO25)
- net IO1 renamed UART0_TX
- net IO3 renamed UART0_RX
- net UART1_RX renamed CAN_RX
- net UART1_TX renamed CAN_TX
- net UART2_RX renamed IO4
- new net CAN_STBY: U1.10 (DAC_1/ADC2_CH8/GPIO25)
Other:
- moved on the sheet: C3, C4
