File: hw/mainBoard/connectors.kicad_sch (KiCad schematic)
At the start: 4 parts, among them J1 Conn_2Rows-39Pins, J2 UART_MODULE, J3 JTAG

Commit message: hw
Parts:
- removed J2: UART_MODULE, symbol Connector_Generic:Conn_01x05
Connections:
- net IO16 renamed UART2_RX
- net IO17 renamed UART2_TX
- net ~{UART_INT} renamed UART1_RX
- net ~{UART_MODULE_CS} renamed UART1_TX
- net ~{UART_MODULE_RST} renamed IO4
Changed lines of the file:
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@@
-    (stroke (width 0) (type default))
-  )
-  (wire (pts (xy 104.14 120.65) (xy 113.03 120.65))
     (stroke (width 0) (type default))
   )
@@
     (stroke (width 0) (type default))
   )
-  (wire (pts (xy 104.14 130.81) (xy 113.03 130.81))
-    (stroke (width 0) (type default))
-  )
   (wire (pts (xy 173.99 119.38) (xy 181.61 119.38))
     (stroke (width 0) (type default))
@@
     (stroke (width 0) (type default))
   )
-  (wire (pts (xy 104.14 123.19) (xy 113.03 123.19))
-    (stroke (width 0) (type default))
-  )
   (wire (pts (xy 154.94 129.54) (xy 161.29 129.54))
     (stroke (width 0) (type default))
@@
     (stroke (width 0) (type default))
   )
-  (wire (pts (xy 104.14 128.27) (xy 113.03 128.27))
-    (stroke (width 0) (type default))
-  )
   (wire (pts (xy 101.6 53.34) (xy 111.76 53.34))
     (stroke (width 0) (type default))
@@
     (stroke (width 0) (type default))
   )
-  (wire (pts (xy 104.14 125.73) (xy 113.03 125.73))
-    (stroke (width 0) (type default))
-  )
   (wire (pts (xy 124.46 68.58) (xy 134.62 68.58))
     (stroke (width 0) (type default))
@@
     )
   )
-  (global_label "MOSI" (shape input) (at 104.14 128.27 180) (fields_autoplaced)
-    (effects (font (size 1.27 1.27)) (justify right))
-    (property "Intersheetrefs" "${INTERSHEET_REFS}" (at 96.8005 128.27 0)
-      (effects (font (size 1.27 1.27)) (justify right) hide)
-    )
-  )
   (global_label "MTDI" (shape input) (at 181.61 127 0) (fields_autoplaced)
     (effects (font (size 1.27 1.27)) (justify left))
@@
     )
   )
-  (global_label "MISO" (shape input) (at 104.14 130.81 180) (fields_autoplaced)
-    (effects (font (size 1.27 1.27)) (justify right))
-    (property "Intersheetrefs" "${INTERSHEET_REFS}" (at 96.8005 130.81 0)
-      (effects (font (size 1.27 1.27)) (justify right) hide)
-    )
-  )
   (global_label "IO12" (shape input) (at 101.6 63.5 180) (fields_autoplaced)
     (effects (font (size 1.27 1.27)) (justify right))
@@
     )
   )
-  (global_label "~{UART_INT}" (shape input) (at 104.14 120.65 180) (fields_autoplaced)
-    (effects (font (size 1.27 1.27)) (justify right))
-    (property "Intersheetrefs" "${INTERSHEET_REFS}" (at 96.8005 120.65 0)
-      (effects (font (size 1.27 1.27)) (justify right) hide)
-    )
-  )
   (global_label "GND" (shape input) (at 134.62 93.98 0) (fields_autoplaced)
     (effects (font (size 1.27 1.27)) (justify left))
@@
     )
   )
-  (global_label "IO17" (shape input) (at 101.6 76.2 180) (fields_autoplaced)
+  (global_label "UART2_TX" (shape input) (at 101.6 76.2 180) (fields_autoplaced)
     (effects (font (size 1.27 1.27)) (justify right))
     (property "Intersheetrefs" "${INTERSHEET_REFS}" (at 94.2605 76.2 0)
@@
     )
   )
-  (global_label "~{UART_MODULE_CS}" (shape input) (at 104.14 123.19 180) (fields_autoplaced)
-    (effects (font (size 1.27 1.27)) (justify right))
-    (property "Intersheetrefs" "${INTERSHEET_REFS}" (at 96.8005 123.19 0)
-      (effects (font (size 1.27 1.27)) (justify right) hide)
-    )
-  )
   (global_label "IO36" (shape input) (at 134.62 88.9 0) (fields_autoplaced)
     (effects (font (size 1.27 1.27)) (justify left))
@@
     )
   )
-  (global_label "~{UART_MODULE_CS}" (shape input) (at 101.6 96.52 180) (fields_autoplaced)
-    (effects (font (size 1.27 1.27)) (justify right))
-    (property "Intersheetrefs" "${INTERSHEET_REFS}" (at 94.2605 96.52 0)
-      (effects (font (size 1.27 1.27)) (justify right) hide)
-    )
-  )
-  (global_label "~{UART_INT}" (shape input) (at 101.6 93.98 180) (fields_autoplaced)
-    (effects (font (size 1.27 1.27)) (justify right))
-    (property "Intersheetrefs" "${INTERSHEET_REFS}" (at 94.2605 93.98 0)
+  (global_label "UART1_TX" (shape input) (at 101.6 96.52 180) (fields_autoplaced)
+    (effects (font (size 1.27 1.27)) (justify right))
+    (property "Intersheetrefs" "${INTERSHEET_REFS}" (at 89.6039 96.52 0)
+      (effects (font (size 1.27 1.27)) (justify right) hide)
+    )
+  )
+  (global_label "UART1_RX" (shape input) (at 101.6 93.98 180) (fields_autoplaced)
+    (effects (font (size 1.27 1.27)) (justify right))
+    (property "Intersheetrefs" "${INTERSHEET_REFS}" (at 89.3015 93.98 0)
       (effects (font (size 1.27 1.27)) (justify right) hide)
     )
@@
     )
   )
-  (global_label "~{UART_MODULE_RST}" (shape input) (at 101.6 58.42 180) (fields_autoplaced)
+  (global_label "IO4" (shape input) (at 101.6 58.42 180) (fields_autoplaced)
     (effects (font (size 1.27 1.27)) (justify right))
     (property "Intersheetrefs" "${INTERSHEET_REFS}" (at 95.47 58.42 0)
@@
     )
   )
-  (global_label "IO16" (shape input) (at 101.6 73.66 180) (fields_autoplaced)
+  (global_label "UART2_RX" (shape input) (at 101.6 73.66 180) (fields_autoplaced)
     (effects (font (size 1.27 1.27)) (justify right))
     (property "Intersheetrefs" "${INTERSHEET_REFS}" (at 94.2605 73.66 0)
@@
     (property "Intersheetrefs" "${INTERSHEET_REFS}" (at 141.9595 81.28 0)
       (effects (font (size 1.27 1.27)) (justify left) hide)
-    )
-  )
-  (global_label "SCLK" (shape input) (at 104.14 125.73 180) (fields_autoplaced)
-    (effects (font (size 1.27 1.27)) (justify right))
-    (property "Intersheetrefs" "${INTERSHEET_REFS}" (at 96.8005 125.73 0)
-      (effects (font (size 1.27 1.27)) (justify right) hide)
     )
   )
@@
         )
       )
-    )
-  )
-  (symbol (lib_id "Connector_Generic:Conn_01x05") (at 118.11 125.73 0) (unit 1)
-    (in_bom yes) (on_board yes) (dnp no)
-    (property "Reference" "J2" (at 116.84 114.3 0)
-      (effects (font (size 1.27 1.27)) (justify left))
-    )
-    (property "Value" "UART_MODULE" (at 111.76 116.84 0)
-      (effects (font (size 1.27 1.27)) (justify left))
-    )
-    (property "Footprint" "" (at 118.11 125.73 0)
-      (effects (font (size 1.27 1.27)) hide)
-    )
-    (property "Datasheet" "~" (at 118.11 125.73 0)
-      (effects (font (size 1.27 1.27)) hide)
-    )
-    (pin "1")
-    (pin "3")
-    (pin "4")
-    (pin "2")
-    (pin "5")
-    (instances
-      (project "mainBoard"
-        (path "/afbe4b5f-4e5c-4a12-a44b-208d158a3f7a/e09778c5-d723-4378-b78b-5054d4eb0fd5"
-          (reference "J2") (unit 1)
-        )
-      )

Commit message: hw + blok schema
Parts:
- removed J1: Conn_2Rows-39Pins, symbol Connector_Generic:Conn_2Rows-39Pins
- added J1: LED strip, symbol Connector_Generic:Conn_01x03
- added J5: Relays_board, Connector_JST:JST_XH_B4B-XH-AM_1x04_P2.50mm_Vertical, symbol Connector_Generic:Conn_01x04
- added J6: Display, Connector_JST:JST_XH_B4B-XH-AM_1x04_P2.50mm_Vertical, symbol Connector_Generic:Conn_01x04
- added J7: POWER SUPLY, symbol Connector:Conn_01x02_Pin
- added J8: Conn_2Rows-33Pins, symbol Connector_Generic:Conn_2Rows-33Pins
- added U3: TXU0101DBVR, SOT-23-6-DBV_TEX, symbol TXU0101:TXU0101DBVR
Connections:
- net 3V3 is gone; now on net GND: JP1.1 (A)
- net EN: now also J8.5 (Pin_5)
- net GND: now also J1.3 (Pin_3), J5.1 (Pin_1), J5.4 (Pin_4), J6.1 (Pin_1), J6.4 (Pin_4), J7.2 (Pin_2), J8.1 (Pin_1), J8.2 (Pin_2), J8.3 (Pin_3), J8.31 (Pin_31), J8.33 (Pin_33), J8.4 (Pin_4), U3.1 (VCCA), U3.2 (GND), U3.5 (OE)
- net IO0: now also J8.6 (Pin_6)
- net IO1: now also J8.8 (Pin_8)
- net IO2: now also J8.10 (Pin_10)
- net IO3: now also J8.12 (Pin_12)
- net IO32: now also J8.15 (Pin_15)
- net IO33: now also J8.17 (Pin_17)
- net IO34: now also J8.19 (Pin_19)
- net IO35: now also J8.21 (Pin_21)
- net IO36: now also J8.23 (Pin_23)
- net IO39: now also J8.25 (Pin_25)
- net IO4: now also J8.14 (Pin_14)
- net IO5: now also J8.16 (Pin_16)
- net MISO: now also J8.24 (Pin_24)
- net MOSI: now also J8.30 (Pin_30)
- net MTCK: now also J8.9 (Pin_9)
- net MTDI: now also J8.7 (Pin_7)
- net MTDO: now also J8.13 (Pin_13)
- net MTMS: now also J8.11 (Pin_11)
- net SCLK: now also J8.22 (Pin_22)
- net UART1_RX: now also J8.27 (Pin_27)
- net UART1_TX: now also J8.29 (Pin_29)
- net UART2_RX: now also J8.18 (Pin_18)
- net UART2_TX: now also J8.20 (Pin_20)
- new net: J1.2 (Pin_2), U3.4 (BY)
- new net 24V: J7.1 (Pin_1)
- new net 5.2V: J1.1 (Pin_1), U3.6 (VCCB)
- new net LED_STRIP: J8.32 (Pin_32), U3.3 (A)
- new net SCL: J5.3 (Pin_3), J6.3 (Pin_3), J8.28 (Pin_28)
- new net SDA: J5.2 (Pin_2), J6.2 (Pin_2), J8.26 (Pin_26)
Other:
- moved on the sheet: J3, JP1

Commit message: nejaky hw + teorie + desky
Changed lines of the file:
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@@
 (kicad_sch (version 20230121) (generator eeschema)
   (paper "A4")
+  (bus_alias "ESP_PINS_1" (members "IO33" "IO36" "IO32" "IO35" "MTDO" "MTCK" "MTMS" "IO34" "IO39" "MTDI" "EN"))
+  (bus_alias "ESP_PINS_2" (members "IO2" "SCL" "IO5" "IO4" "IO1" "SDA" "MISO" "MOSI" "IO0" "UART1_RX" "UART1_TX" "UART2_RX" "UART2_TX" "SCLK" "IO3" "LED_STRIP"))
+  (bus_alias "I2C" (members "SDA" "SCL"))
+  (bus_alias "JTAG" (members "MTMS" "MTCK" "MTDO" "MTDI"))
   (junction (at 111.76 30.48) (diameter 0) (color 0 0 0 0)
   )
@@
     (effects (font (size 1.27 1.27)) (justify right))
   )
-  (hierarchical_label "I2C" (shape bidirectional) (at 114.3 73.66 180) (fields_autoplaced)
+  (hierarchical_label "{I2C}" (shape bidirectional) (at 114.3 73.66 180) (fields_autoplaced)
     (effects (font (size 1.27 1.27)) (justify right))
   )
@@
     (effects (font (size 1.27 1.27)) (justify right))
   )
-  (hierarchical_label "JTAG" (shape bidirectional) (at 147.32 38.1 0) (fields_autoplaced)
+  (hierarchical_label "{JTAG}" (shape bidirectional) (at 147.32 38.1 0) (fields_autoplaced)
     (effects (font (size 1.27 1.27)) (justify left))
   )
@@
     (effects (font (size 1.27 1.27)) (justify right))
   )
-  (hierarchical_label "ESP_PINS_1" (shape bidirectional) (at 91.44 127 0) (fields_autoplaced)
+  (hierarchical_label "{ESP_PINS_1}" (shape bidirectional) (at 91.44 127 0) (fields_autoplaced)
     (effects (font (size 1.27 1.27)) (justify left))
   )
@@
     (effects (font (size 1.27 1.27)) (justify right))
   )
-  (hierarchical_label "ESP_PINS_2" (shape bidirectional) (at 91.44 119.38 0) (fields_autoplaced)
+  (hierarchical_label "{ESP_PINS_2}" (shape bidirectional) (at 91.44 119.38 0) (fields_autoplaced)
     (effects (font (size 1.27 1.27)) (justify left))
   )

Commit message: hw - changed uart2 pins, latex- ridici jednotka
Connections:
- net IO4 is gone; now on net UART2_RX: J8.14 (Pin_14)
- net UART2_RX: no longer J8.18 (Pin_18)
- new net IO16: J8.18 (Pin_18)
Other:
- moved on the sheet: J1, J3, J5, J6, J7, J8, JP1, U3

Commit message: drawing layout
Parts:
- removed J8: Conn_2Rows-33Pins, symbol Connector_Generic:Conn_2Rows-33Pins
- added C13, C14: 0.1uF, Capacitor_SMD:C_1206_3216Metric_Pad1.33x1.80mm_HandSolder, symbol Device:C
- added J8: Conn_02x16_Odd_Even, Connector_PinHeader_2.54mm:PinHeader_2x16_P2.54mm_Vertical, symbol Connector_Generic:Conn_02x16_Odd_Even
- J1: footprint (none) -> Connector_JST:JST_EH_B3B-EH-A_1x03_P2.50mm_Vertical
- J3: footprint (none) -> Connector_PinHeader_1.27mm:PinHeader_2x05_P1.27mm_Vertical; symbol Connector_Generic:Conn_2Rows-09Pins -> Connector_Generic:Conn_02x05_Odd_Even
- J7: footprint (none) -> TerminalBlock:TerminalBlock_Altech_AK300-2_P5.00mm
- JP1: footprint (none) -> TestPoint:TestPoint_2Pads_Pitch2.54mm_Drill0.8mm
- U3: footprint SOT-23-6-DBV_TEX -> TXU0101:SOT-23-6-DBV_TEX
Connections:
- net 5.2V: now also C13.1
- net EN: now also J8.5 (Pin_5)
- net GND: now also C13.2, C14.2, J8.3 (Pin_3), J8.31 (Pin_31), J8.4 (Pin_4); no longer J5.1 (Pin_1), J6.1 (Pin_1), JP1.1 (A), U3.1 (VCCA), U3.5 (OE)
- net IO0: now also J8.6 (Pin_6)
- net IO16: now also J8.18 (Pin_18)
- net IO2: now also J8.10 (Pin_10)
- net IO32: now also J8.15 (Pin_15)
- net IO33: now also J8.17 (Pin_17)
- net IO34: now also J8.19 (Pin_19)
- net IO35: now also J8.21 (Pin_21)
- net IO36: now also J8.23 (Pin_23)
- net IO39: now also J8.25 (Pin_25)
- net IO5: now also J8.16 (Pin_16)
- net LED_STRIP: now also J8.20 (Pin_20)
- net MISO: now also J8.24 (Pin_24)
- net MOSI: now also J8.30 (Pin_30)
- net MTCK: now also J8.9 (Pin_9)
- net MTDI: now also J8.7 (Pin_7)
- net MTDO: now also J8.13 (Pin_13)
- net MTMS: now also J8.11 (Pin_11)
- net SCL: now also J8.28 (Pin_28)
- net SCLK: now also J8.22 (Pin_22)
- net SDA: now also J8.26 (Pin_26)
- new net 3V3: C14.1, J5.1 (Pin_1), J6.1 (Pin_1), J8.1 (Pin_1), J8.2 (Pin_2), JP1.1 (A), U3.1 (VCCA), U3.5 (OE)
- new net CAN_RX: J8.27 (Pin_27)
- new net CAN_STBY: J8.32 (Pin_32)
- new net CAN_TX: J8.29 (Pin_29)
- new net IO4: J8.14 (Pin_14)
- new net UART0_RX: J8.12 (Pin_12)
- new net UART0_TX: J8.8 (Pin_8)
- no-connect marks 0 -> 1

Commit message: finale bez rybicky
Parts:
- renumbered C13 to C19, C14 to C20, J6 to J3, J1 to J4, J3 to J6
Changed lines of the file:
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@@
   (symbol (lib_id "Connector_Generic:Conn_01x04") (at 180.34 88.9 0) (unit 1)
     (in_bom yes) (on_board yes) (dnp no) (fields_autoplaced)
-    (property "Reference" "J6" (at 182.88 88.9 0)
+    (property "Reference" "J3" (at 182.88 88.9 0)
       (effects (font (size 1.27 1.27)) (justify left))
     )
@@
       (project "mainBoard"
         (path "/afbe4b5f-4e5c-4a12-a44b-208d158a3f7a/e09778c5-d723-4378-b78b-5054d4eb0fd5"
-          (reference "J6") (unit 1)
+          (reference "J3") (unit 1)
         )
       )
@@
   (symbol (lib_id "Connector_Generic:Conn_02x05_Odd_Even") (at 158.75 40.64 0) (unit 1)
     (in_bom yes) (on_board yes) (dnp no) (fields_autoplaced)
-    (property "Reference" "J3" (at 160.02 29.21 0)
+    (property "Reference" "J6" (at 160.02 29.21 0)
       (effects (font (size 1.27 1.27)))
     )
@@
       (project "mainBoard"
         (path "/afbe4b5f-4e5c-4a12-a44b-208d158a3f7a/e09778c5-d723-4378-b78b-5054d4eb0fd5"
-          (reference "J3") (unit 1)
+          (reference "J6") (unit 1)
         )
       )
@@
   (symbol (lib_id "Device:C") (at 203.2 138.43 0) (unit 1)
     (in_bom yes) (on_board yes) (dnp no)
-    (property "Reference" "C14" (at 205.74 138.43 0)
+    (property "Reference" "C20" (at 205.74 138.43 0)
       (effects (font (size 1.27 1.27)) (justify left))
     )
@@
       (project "mainBoard"
         (path "/afbe4b5f-4e5c-4a12-a44b-208d158a3f7a/e09778c5-d723-4378-b78b-5054d4eb0fd5"
-          (reference "C14") (unit 1)
+          (reference "C20") (unit 1)
         )
       )
@@
   (symbol (lib_id "Device:C") (at 193.04 138.43 0) (unit 1)
     (in_bom yes) (on_board yes) (dnp no)
-    (property "Reference" "C13" (at 195.58 138.43 0)
+    (property "Reference" "C19" (at 195.58 138.43 0)
       (effects (font (size 1.27 1.27)) (justify left))
     )
@@
       (project "mainBoard"
         (path "/afbe4b5f-4e5c-4a12-a44b-208d158a3f7a/e09778c5-d723-4378-b78b-5054d4eb0fd5"
-          (reference "C13") (unit 1)
+          (reference "C19") (unit 1)
         )
       )
@@
   (symbol (lib_id "Connector_Generic:Conn_01x03") (at 241.3 121.92 0) (unit 1)
     (in_bom yes) (on_board yes) (dnp no)
-    (property "Reference" "J1" (at 243.84 120.65 0)
+    (property "Reference" "J4" (at 243.84 120.65 0)
       (effects (font (size 1.27 1.27)) (justify left))
     )
@@
       (project "mainBoard"
         (path "/afbe4b5f-4e5c-4a12-a44b-208d158a3f7a/e09778c5-d723-4378-b78b-5054d4eb0fd5"
-          (reference "J1") (unit 1)
-        )
-      )
+          (reference "J4") (unit 1)
+        )
+      )
