File: hw/mainBoard/mainBoard.kicad_pcb (KiCad board)
At the start: 4 copper layers, 50 x 94.2 mm, 65 parts, among them IC1 ATA6561-GAQW-N, J1 G17C0900132EU, J2 G17C0900132EU, J3 Display, J4 LED strip, J5 Relays_board, J6 JTAG, J7 POWER SUPLY, J8 Conn_02x16_Odd_Even, Q1 NMOS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

Commit message: gerbere s rybou
Parts:
- added RYBA: LOGO, LOGO, F.Cu at (151.3, 82.1)
Routing:
- net GND: vias 98 -> 99
Other:
- board text added: "JLCJLCJLCJLC"
