File: hw/mainBoard/power_suply.kicad_sch (KiCad schematic)
At the start: 29 parts, among them Q1 NMOS, Q2 NMOS, U4 LM5148RGYR

Commit message: oprava schematicu
Other:
- note added: "V_FB = 0.8V = V_out*R7/(R7+R8) => R8=54.9kOhm (Datasheet sec. 8.3.8)"
- note removed: "V_FB = 0.8V = V_out*R15/(R15+R16) => R16=54.9kOhm (Datasheet sec. 8.3.8)"
Changed lines of the file:
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@@
     (effects (font (size 1.27 1.27)) (justify left bottom))
   )
-  (text "V_FB = 0.8V \n      = V_out*R15/(R15+R16)\n	 => R16=54.9kOhm\n(Datasheet sec. 8.3.8)"
+  (text "V_FB = 0.8V \n      = V_out*R7/(R7+R8)\n	 => R8=54.9kOhm\n(Datasheet sec. 8.3.8)"
     (at 95.25 147.32 0)
     (effects (font (size 1.27 1.27)) (justify left bottom))
