File: hw/peripherialModule/peripherialModule.kicad_pcb (KiCad board)
At the start: 2 copper layers, 34.2 x 53.2 mm, 20 parts, among them IC1 ATA6561-GAQW-N, J1 Conn_01x13_Socket, J2 Conn_01x13_Socket, J3 G17C0900132EU, J4 G17C0900132EU, J5 Conn_01x03_Socket, J6 726386-2, J7 726386-2, SW1 SW_Push, U1 TLV76133DCYR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

Commit message: boards are changing
Parts:
- removed J2: Conn_01x13_Socket, Connector_PinSocket_2.54mm:PinSocket_1x13_P2.54mm_Vertical
- removed J7: 726386-2, FASTON:726386-2
- added G***: LOGO, LOGO, F.Cu at (230.3, 90.8)
- added J8: Conn_01x05_Socket, Connector_PinSocket_2.54mm:PinSocket_1x05_P2.54mm_Vertical, F.Cu at (233.7, 70.0)
- added J9: Conn_01x03_Socket, Connector_PinSocket_2.54mm:PinSocket_1x03_P2.54mm_Vertical, F.Cu at (218.4, 90.3)
- added REF**: MountingHole_2.2mm_M2_Pad, MountingHole:MountingHole_2.2mm_M2_Pad, F.Cu at (260.1, 107.0)
- J1: value Conn_01x13_Socket -> Conn_02x11_Socket; footprint Connector_PinSocket_2.54mm:PinSocket_1x13_P2.54mm_Vertical -> Connector_PinSocket_2.54mm:PinSocket_2x11_P2.54mm_Vertical
- J6: value 726386-2 -> Conn_01x03_Socket; footprint FASTON:726386-2 -> Connector_PinSocket_2.54mm:PinSocket_1x03_P2.54mm_Vertical
- R2: value 100 -> 1k
- moved J6 53.9 mm to (223.5, 90.3), turned to 0 degrees
- moved J5 45.7 mm to (231.1, 75.1)
- moved C3 38.9 mm to (225.1, 69.0)
- moved C4 38.9 mm to (209.9, 68.3)
- moved C5 38.9 mm to (223.6, 72.5)
- moved JP1 38.9 mm to (226.4, 71.6)
- moved R1 38.9 mm to (211.3, 74.9)
- moved R2 38.9 mm to (208.5, 74.9)
- moved SW1 38.9 mm to (209.9, 71.4)
- moved U1 38.9 mm to (218.2, 71.4)
- moved J1 38.1 mm to (203.2, 70.0)
- moved C6 37.4 mm to (225.6, 82.4)
- moved U2 37.4 mm to (217.7, 82.2)
- moved J4 37.2 mm to (222.6, 100.3)
- moved J3 36.9 mm to (211.5, 64.8)
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Connections:
- J1 pad 1: /5.2V -> GND
- J1 pad 10: /RA4 -> /RA1
- J1 pad 11: /RA5 -> /RC5
- J1 pad 12: /RA6 -> /RA2
- J1 pad 13: /RA7 -> /RC4
- J1 pad 2: /5.2V -> GND
- J1 pad 3: GND -> /5.2V
- J1 pad 4: /VDD -> /5.2V
- J1 pad 6: /RA0 -> /VDD
- J1 pad 7: /RA1 -> /RC7
- J1 pad 8: /RA2 -> /RA0
- J1 pad 9: /RA3 -> /RC6
- J6 pad 1: /24V -> GND
- J6 pad 2: /24V -> GND
Routing:
- net /5.2V: track 114.3 -> 21.1 mm, vias 3 -> 4
- net /24V: track 58.0 -> 0.00 mm
- net /VDD: track 61.5 -> 48.4 mm, vias 4 -> 7
- net /RC0: track 24.3 -> 12.3 mm, vias 0 -> 1
- net /CAN_TX: track 25.3 -> 14.9 mm, vias 2 -> 0
- net /RC1: track 23.4 -> 13.0 mm, vias 0 -> 1
- net /RC2: track 23.7 -> 13.8 mm, vias 0 -> 1
- net /RB5: track 20.1 -> 10.2 mm
- net /RC3: track 24.5 -> 14.7 mm, vias 0 -> 1
- net /RA6: track 29.7 -> 20.1 mm
- net Net-(IC1-CANL): track 42.5 -> 51.8 mm, vias 1 -> 0
- net Net-(IC1-CANH): track 42.0 -> 50.9 mm
- net /RC7: track 12.5 -> 21.0 mm, vias 0 -> 1
- net /RC6: track 11.7 -> 20.1 mm, vias 0 -> 1
- net /CAN_STBY: track 26.1 -> 19.0 mm, vias 2 -> 0
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- added copper zone on In2.Cu, net /24V
- added copper zone on In2.Cu, net /3V3
- added copper zone on In2.Cu, net /5.2V
- added copper zone on In2.Cu, net /VDD
- added copper zone on In1.Cu, net GND
Other:
- board size 34.2 x 53.2 mm -> 37 x 50 mm
- copper layers 2 -> 4
- board text added: "2024 Jakub Charvot, FEKT VUT"
- board text added: "3.3V"
- board text added: "5.2V"
- board text added: "GND"
- board text added: "RC0 RA4"
- board text added: "RC1 RA5"
- board text added: "RC2 RA6"
- board text added: "RC3 RA7"
- board text added: "RC4 RA3"
- board text added: "RC5 RA2"
- board text added: "RC6 RA1"
- board text added: "RC7 RA0"

Commit message: hw - ledBoard
Parts:
- removed REF**: MountingHole_2.2mm_M2_Pad, MountingHole:MountingHole_2.2mm_M2_Pad
- C4, C6: value 0.1u -> 0.1uF
- SW1: moved to B.Cu
- moved R2 3.37 mm to (208.3, 71.6)
- moved R1 3.32 mm to (211.4, 71.6)
- moved SW1 2.86 mm to (209.9, 68.5)
Routing:
- net /24V: track 0.00 -> 5.08 mm
- net /VDD: track 48.4 -> 51.3 mm
- net Net-(C4-Pad1): track 8.58 -> 5.66 mm, vias 0 -> 1
- net GND: track 30.1 -> 31.0 mm, vias 17 -> 18
- net /~{MCLR}: track 32.4 -> 33.0 mm
Other:
- board text added: "+24V"
- board text added: "ICSP"
- board text added: "JLCJLCJLCJLC"
- board text added: "RB0"
- board text added: "RB1"
- board text added: "RB5"
